File: PCB/matrix.sch (KiCad schematic (older format))
At the start: 134 parts, among them K1 MX-NoLED, K10 MX-NoLED, K11 MX-NoLED, K12 MX-NoLED, K13 MX-NoLED, K14 MX-NoLED, K15 MX-NoLED, K16 MX-NoLED, K17 MX-NoLED, K18 MX-NoLED, K19 MX-NoLED, K2 MX-NoLED, K20 MX-NoLED, K21 MX-NoLED, K22 MX-NoLED, K23 MX-NoLED, K24 MX-NoLED, K25 MX-NoLED, K26 MX-NoLED, K27 MX-NoLED, K28 MX-NoLED, K29 MX-NoLED, K3 MX-NoLED, K30 MX-NoLED, K31 MX-NoLED, K32 MX-NoLED, K33 MX-NoLED, K34 MX-NoLED, K35 MX-NoLED, K36 MX-NoLED, K37 MX-NoLED, K38 MX-NoLED, K39 MX-NoLED, K4 MX-NoLED, K40 MX-NoLED, K41 MX-NoLED, K42 MX-NoLED, K43 MX-NoLED, K44 MX-NoLED, K45 MX-NoLED, K46 MX-NoLED, K47 MX-NoLED, K48 MX-NoLED, K49 MX-NoLED, K5 MX-NoLED, K50 MX-NoLED, K51 MX-NoLED, K52 MX-NoLED, K53 MX-NoLED, K54 MX-NoLED, K55 MX-NoLED, K56 MX-NoLED, K57 MX-NoLED, K58 MX-NoLED, K59 MX-NoLED, K6 MX-NoLED, K60 MX-NoLED, K61 MX-NoLED, K62 MX-NoLED, K63 MX-NoLED, K64 MX-NoLED, K65 MX-NoLED, K66 MX-NoLED, K67 MX-NoLED, K7 MX-NoLED, K8 MX-NoLED, K9 MX-NoLED

Commit message: pcb alignment
Parts:
- K1: value MX-NoLED -> Esc
- K10: value MX-NoLED -> #9
- K11: value MX-NoLED -> #0
- K12: value MX-NoLED -> -
- K13: value MX-NoLED -> =
- K14: value MX-NoLED -> BckSpc
- K15: value MX-NoLED -> Del
- K16: value MX-NoLED -> Tab
- K17: value MX-NoLED -> Q
- K18: value MX-NoLED -> W
- K19: value MX-NoLED -> E
- K2: value MX-NoLED -> #1
- K20: value MX-NoLED -> R
- K21: value MX-NoLED -> T
- K22: value MX-NoLED -> Y
- K23: value MX-NoLED -> U
- K24: value MX-NoLED -> I
- K25: value MX-NoLED -> O
- K26: value MX-NoLED -> P
- K27: value MX-NoLED -> [
- K28: value MX-NoLED -> ]
- K29: value MX-NoLED -> |\\
- K3: value MX-NoLED -> #2
- K30: value MX-NoLED -> PgUp
- K31: value MX-NoLED -> CpsLck
- K32: value MX-NoLED -> A
- K33: value MX-NoLED -> S
- K34: value MX-NoLED -> D
- K35: value MX-NoLED -> F
- K36: value MX-NoLED -> G
- K37: value MX-NoLED -> H
- K38: value MX-NoLED -> J
- K39: value MX-NoLED -> K
- K4: value MX-NoLED -> #3
- K40: value MX-NoLED -> L
- K41: value MX-NoLED -> ;
- K42: value MX-NoLED -> '
- K43: value MX-NoLED -> Entr
- K44: value MX-NoLED -> PgDn
- K45: value MX-NoLED -> l_shft
- K46: value MX-NoLED -> Z
- K47: value MX-NoLED -> X
- K48: value MX-NoLED -> C
- K49: value MX-NoLED -> V
- K5: value MX-NoLED -> #4
- K50: value MX-NoLED -> B
- K51: value MX-NoLED -> N
- K52: value MX-NoLED -> M
- K53: value MX-NoLED -> ,
- K54: value MX-NoLED -> .
- K55: value MX-NoLED -> /
- K56: value MX-NoLED -> r_shft
- K57: value MX-NoLED -> up
- K58: value MX-NoLED -> PrntScrn
- K59: value MX-NoLED -> l_ctrl
- K6: value MX-NoLED -> #5
- K60: value MX-NoLED -> win
- K61: value MX-NoLED -> l_alt
- K62: value MX-NoLED -> space
- K63: value MX-NoLED -> r_alt
- K64: value MX-NoLED -> r_ctrl
- K65: value MX-NoLED -> left
- K66: value MX-NoLED -> down
- K67: value MX-NoLED -> right
- K7: value MX-NoLED -> #6
- K8: value MX-NoLED -> #7
- K9: value MX-NoLED -> #8
Other:
- moved on the sheet: D1, D10, D11, D12, D13, D14, D15, D16, D17, D18, D19, D2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
