File: PCB/PCB.kicad_pcb (KiCad board)
At the start: 2 copper layers, 154 parts, among them J1 AVR-ISP-6, K1 MX-NoLED, K10 MX-NoLED, K11 MX-NoLED, K12 MX-NoLED, K13 MX-NoLED, K14 MX-NoLED, K15 MX-NoLED, K16 MX-NoLED, K17 MX-NoLED, K18 MX-NoLED, K19 MX-NoLED, K2 MX-NoLED, K20 MX-NoLED, K21 MX-NoLED, K22 MX-NoLED, K23 MX-NoLED, K24 MX-NoLED, K25 MX-NoLED, K26 MX-NoLED, K27 MX-NoLED, K28 MX-NoLED, K29 MX-NoLED, K3 MX-NoLED, K30 MX-NoLED, K31 MX-NoLED, K32 MX-NoLED, K33 MX-NoLED, K34 MX-NoLED, K35 MX-NoLED, K36 MX-NoLED, K37 MX-NoLED, K38 MX-NoLED, K39 MX-NoLED, K4 MX-NoLED, K40 MX-NoLED, K41 MX-NoLED, K42 MX-NoLED, K43 MX-NoLED, K44 MX-NoLED, K45 MX-NoLED, K46 MX-NoLED, K47 MX-NoLED, K48 MX-NoLED, K49 MX-NoLED, K5 MX-NoLED, K50 MX-NoLED, K51 MX-NoLED, K52 MX-NoLED, K53 MX-NoLED, K54 MX-NoLED, K55 MX-NoLED, K56 MX-NoLED, K57 MX-NoLED, K58 MX-NoLED, K59 MX-NoLED, K6 MX-NoLED, K60 MX-NoLED, K61 MX-NoLED, K62 MX-NoLED, K63 MX-NoLED, K64 MX-NoLED, K65 MX-NoLED, K66 MX-NoLED, K67 MX-NoLED, K7 MX-NoLED, K8 MX-NoLED, K9 MX-NoLED, SW1 SW_Push

Commit message: pcb alignment
Parts:
- K1: value MX-NoLED -> Esc
- K10: value MX-NoLED -> #9
- K11: value MX-NoLED -> #0
- K12: value MX-NoLED -> -
- K13: value MX-NoLED -> =
- K14: value MX-NoLED -> BckSpc
- K15: value MX-NoLED -> Del
- K16: value MX-NoLED -> Tab
- K17: value MX-NoLED -> Q
- K18: value MX-NoLED -> W
- K19: value MX-NoLED -> E
- K2: value MX-NoLED -> #1
- K20: value MX-NoLED -> R
- K21: value MX-NoLED -> T
- K22: value MX-NoLED -> Y
- K23: value MX-NoLED -> U
- K24: value MX-NoLED -> I
- K25: value MX-NoLED -> O
- K26: value MX-NoLED -> P
- K27: value MX-NoLED -> [
- K28: value MX-NoLED -> ]
- K29: value MX-NoLED -> |\
- K3: value MX-NoLED -> #2
- K30: value MX-NoLED -> PgUp
- K31: value MX-NoLED -> CpsLck
- K32: value MX-NoLED -> A
- K33: value MX-NoLED -> S
- K34: value MX-NoLED -> D
- K35: value MX-NoLED -> F
- K36: value MX-NoLED -> G
- K37: value MX-NoLED -> H
- K38: value MX-NoLED -> J
- K39: value MX-NoLED -> K
- K4: value MX-NoLED -> #3
- K40: value MX-NoLED -> L
- K41: value MX-NoLED -> ;
- K42: value MX-NoLED -> '
- K43: value MX-NoLED -> Entr
- K44: value MX-NoLED -> PgDn
- K45: value MX-NoLED -> l_shft
- K46: value MX-NoLED -> Z
- K47: value MX-NoLED -> X
- K48: value MX-NoLED -> C
- K49: value MX-NoLED -> V
- K5: value MX-NoLED -> #4
- K50: value MX-NoLED -> B
- K51: value MX-NoLED -> N
- K52: value MX-NoLED -> M
- K53: value MX-NoLED -> ,
- K54: value MX-NoLED -> .
- K55: value MX-NoLED -> /
- K56: value MX-NoLED -> r_shft
- K57: value MX-NoLED -> up
- K58: value MX-NoLED -> PrntScrn
- K59: value MX-NoLED -> l_ctrl
- K6: value MX-NoLED -> #5
- K60: value MX-NoLED -> win
- K61: value MX-NoLED -> l_alt
- K62: value MX-NoLED -> space
- K63: value MX-NoLED -> r_alt
- K64: value MX-NoLED -> r_ctrl
- K65: value MX-NoLED -> left
- K66: value MX-NoLED -> down
- K67: value MX-NoLED -> right
- K7: value MX-NoLED -> #6
- K8: value MX-NoLED -> #7
- K9: value MX-NoLED -> #8
- moved K17 462.8 mm to (61.9, 52.4)
- moved K19 452.9 mm to (100.0, 52.4)
- moved K18 425.3 mm to (81.0, 52.4)
- moved K60 424.6 mm to (59.5, 109.5)
- moved K45 401.1 mm to (45.2, 90.5)
- moved K33 400.5 mm to (85.7, 71.4)
- moved K3 395.2 mm to (71.4, 33.3)
- moved K22 381.6 mm to (157.2, 52.4)
- moved K6 378.0 mm to (128.6, 33.3)
- moved K32 377.6 mm to (66.7, 71.4)
- moved D30 371.2 mm to (325.4, 57.1), turned to 270 degrees
- moved K36 370.9 mm to (142.9, 71.4)
- moved K1 370.4 mm to (33.3, 33.3), turned to 180 degrees
- moved K20 365.5 mm to (119.1, 52.4)
- moved K8 360.6 mm to (166.7, 33.3)
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Connections:
- 32U4 pad 15: +5V -> GND
- 32U4 pad 23: +5V -> GND
- 32U4 pad 35: +5V -> GND
- 32U4 pad 43: +5V -> GND
- 32U4 pad 5: +5V -> GND
- C1-1 pad 2: +5V -> GND
- C2-0.1 pad 1: +5V -> GND
- C3-0.1 pad 1: +5V -> GND
- C4-0.1 pad 1: +5V -> GND
- C5-10 pad 1: +5V -> GND
- C6-22 pad 2: +5V -> GND
- C7-22 pad 2: +5V -> GND
- J1 pad 6: +5V -> GND
- R5-5.1 pad 2: +5V -> GND
- R6-5.1 pad 2: +5V -> GND
- SW1 pad 1: +5V -> GND
- USB-C1 pad 1: +5V -> GND
- USB-C1 pad 12: +5V -> GND
- USB-C1 pad 13: +5V -> GND
- Xtal1 pad 2: +5V -> GND
- Xtal1 pad 4: +5V -> GND
- esd1 pad 1: +5V -> GND

Commit message: switch matrix routing
Parts:
- moved SW1 85.8 mm to (211.1, 108.7), turned to 90 degrees
- moved R2-22 5.02 mm to (169.9, 97.6)
- moved C1-1 4.83 mm to (165.1, 104.0)
- moved R3-22 1.59 mm to (169.9, 100.8)
Routing:
- net row0: track 0.00 -> 362.5 mm, vias 0 -> 16
- net row1: track 0.00 -> 338.2 mm, vias 0 -> 15
- net row4: track 0.00 -> 290.0 mm, vias 0 -> 3
- net row3: track 0.00 -> 289.8 mm, vias 0 -> 9
- net row2: track 0.00 -> 258.3 mm, vias 0 -> 12
- net D+: track 0.00 -> 195.5 mm
- net D-: track 0.00 -> 194.8 mm
- net col10: track 0.00 -> 101.0 mm
- net col11: track 0.00 -> 98.2 mm
- net col2: track 0.00 -> 92.4 mm, vias 0 -> 2
- net col5: track 0.00 -> 90.5 mm, vias 0 -> 2
- net col1: track 0.00 -> 88.2 mm, vias 0 -> 2
- net col13: track 0.00 -> 86.1 mm
- net col12: track 0.00 -> 84.1 mm
- net col0: track 0.00 -> 81.9 mm
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Other:
- board outline added: 304.8 x 99.2 mm

Commit message: PCB Done
Parts:
- added FB1: 60, Inductor_SMD:L_0805_2012Metric_Pad1.05x1.20mm_HandSolder, B.Cu at (50.8, 25.4)
- added G***: LOGO, Graphics:Switch_keeb, F.Cu at (112.7, 108.0)
- moved J1 81.2 mm to (217.5, 100.8), turned to 90 degrees
- moved C1-1 14.3 mm to (178.6, 99.2)
- moved C5-10 14.3 mm to (165.9, 104.0)
- moved R4-10 7.20 mm to (183.6, 100.0), turned to 0 degrees
- moved C7-22 4.49 mm to (193.7, 107.2)
- moved C6-22 3.97 mm to (193.7, 110.3)
- moved C3-0.1 2.74 mm to (183.6, 116.7)
- moved C2-0.1 1.77 mm to (188.1, 104.0)
- moved Xtal1 1.59 mm to (188.9, 108.7), turned to 90 degrees
Connections:
- 32U4 pad 11: MISO -> SCK
- 32U4 pad 36: col6 -> col5
- 32U4 pad 37: col5 -> col6
- 32U4 pad 38: row1 -> row4
- 32U4 pad 39: row4 -> row3
- 32U4 pad 40: row3 -> row2
- 32U4 pad 41: row2 -> row1
- 32U4 pad 9: SCK -> MISO
- R1-10 pad 1: +5V -> GND
- USB-C1 pad 13: GND -> Earth
Routing:
- net GND: track 0.00 -> 374.8 mm, vias 0 -> 49
- net +5V: track 0.00 -> 338.5 mm, vias 0 -> 6
- net row2: track 258.3 -> 543.5 mm, vias 12 -> 16
- net row0: track 362.5 -> 612.0 mm, vias 16 -> 18
- net row1: track 338.2 -> 574.8 mm, vias 15 -> 17
- net row3: track 289.8 -> 453.5 mm, vias 9 -> 11
- net col0: track 81.9 -> 241.6 mm
- net col14: track 76.2 -> 223.1 mm, vias 0 -> 2
- net col1: track 88.2 -> 224.2 mm, vias 2 -> 4
- net col13: track 86.1 -> 212.0 mm, vias 0 -> 2
- net col2: track 92.4 -> 203.0 mm, vias 2 -> 5
- net col12: track 84.1 -> 182.3 mm
- net col3: track 67.0 -> 154.2 mm, vias 0 -> 2
- net col11: track 98.2 -> 171.3 mm, vias 0 -> 2
- net col4: track 67.0 -> 138.2 mm, vias 0 -> 2
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- added copper zone on B.Cu, net Earth
- added copper zone on F.Cu, net Earth
- added copper zone on B.Cu, net GND
- added copper zone on F.Cu, net GND
Other:
- board size 304.8 x 99.2 mm -> 304.8 x 106.4 mm
- board text added: "Designed By: Geraldus Tommy"
- board text added: "Hotswap"
- board text added: "Rev 0"
- board text added: "TOM67"
