File: PCB/PCB.sch (KiCad schematic (older format))
At the start: 20 parts

Commit message: Schemantics
Parts:
- C1-1, C2-0.1, C3-0.1, C4-0.1, C5-10, C6-22, C7-22: footprint (none) -> Capacitor_SMD:C_0805_2012Metric_Pad1.18x1.45mm_HandSolder
- F1: renamed from F; footprint (none) -> Fuse:Fuse_1206_3216Metric_Pad1.42x1.75mm_HandSolder
- J1: renamed from J?; footprint (none) -> random-keyboard-parts:Reset_Pretty
- R1-10, R2-22, R3-22, R4-10, R5-5.1, R6-5.1: footprint (none) -> Resistor_SMD:R_0805_2012Metric_Pad1.20x1.40mm_HandSolder
- SW1: renamed from SW?; footprint (none) -> Button_Switch_SMD:SW_SPST_TL3342
- USB-C1: renamed from USB?; footprint (none) -> Type-C:HRO-TYPE-C-31-M-12-HandSoldering
- Xtal1: renamed from Y?; footprint (none) -> Crystal:Crystal_SMD_3225-4Pin_3.2x2.5mm
- esd1: renamed from U?; footprint (none) -> random-keyboard-parts:SOT143B
- gave numbers to parts that had none: 1
Connections:
- net RESET: now also 32U4.13 (~RESET), R4-10.2, SW1.2
- net row0: now reaches 32U4.1 (PE6)
- net col8: now reaches 32U4.19 (PD1)
- net col9: now reaches 32U4.20 (PD2)
- net col10: now reaches 32U4.21 (PD3)
- net col12: now reaches 32U4.22 (PD5)
- net col11: now reaches 32U4.25 (PD4)
- net col13: now reaches 32U4.26 (PD6)
- net col14: now reaches 32U4.27 (PD7)
- net col0: now reaches 32U4.28 (PB4)
- net col1: now reaches 32U4.29 (PB5)
- net col2: now reaches 32U4.30 (PB6)
- net col3: now reaches 32U4.31 (PC6)
- net col4: now reaches 32U4.32 (PC7)
- net col6: now reaches 32U4.36 (PF7)
- net col5: now reaches 32U4.37 (PF6)
- net row1: now reaches 32U4.38 (PF5)
- net row4: now reaches 32U4.39 (PF4)
- net row3: now reaches 32U4.40 (PF1)
- net row2: now reaches 32U4.41 (PF0)
- net col7: now reaches 32U4.8 (PB0)
- no-connect marks 4 -> 5
Changed lines of the file:
@@
 F 0 "R1-10" V 4404 4250 50  0000 C CNN
 F 1 "10k" V 4495 4250 50  0000 C CNN
-F 2 "" H 4600 4250 50  0001 C CNN
+F 2 "Resistor_SMD:R_0805_2012Metric_Pad1.20x1.40mm_HandSolder" H 4600 4250 50  0001 C CNN
 F 3 "~" H 4600 4250 50  0001 C CNN
 	1    4600 4250
@@
 F 0 "R2-22" V 2354 3150 50  0000 C CNN
 F 1 "22" V 2445 3150 50  0000 C CNN
-F 2 "" H 2550 3150 50  0001 C CNN
+F 2 "Resistor_SMD:R_0805_2012Metric_Pad1.20x1.40mm_HandSolder" H 2550 3150 50  0001 C CNN
 F 3 "~" H 2550 3150 50  0001 C CNN
 	1    2550 3150
@@
 F 0 "R3-22" V 1904 3250 50  0000 C CNN
 F 1 "22" V 1995 3250 50  0000 C CNN
-F 2 "" H 2100 3250 50  0001 C CNN
+F 2 "Resistor_SMD:R_0805_2012Metric_Pad1.20x1.40mm_HandSolder" H 2100 3250 50  0001 C CNN
 F 3 "~" H 2100 3250 50  0001 C CNN
 	1    2100 3250
@@
 F 0 "C1-1" H 2442 3596 50  0000 L CNN
 F 1 "1uF" H 2442 3505 50  0000 L CNN
-F 2 "" H 2350 3550 50  0001 C CNN
+F 2 "Capacitor_SMD:C_0805_2012Metric_Pad1.18x1.45mm_HandSolder" H 2350 3550 50  0001 C CNN
 F 3 "~" H 2350 3550 50  0001 C CNN
 	1    2350 3550
@@
 F 0 "C2-0.1" H 7858 3104 50  0000 R CNN
 F 1 "0.1uF" H 7858 3195 50  0000 R CNN
-F 2 "" H 7950 3150 50  0001 C CNN
+F 2 "Capacitor_SMD:C_0805_2012Metric_Pad1.18x1.45mm_HandSolder" H 7950 3150 50  0001 C CNN
 F 3 "~" H 7950 3150 50  0001 C CNN
 	1    7950 3150
@@
 F 0 "C3-0.1" H 8208 3104 50  0000 R CNN
 F 1 "0.1uF" H 8208 3195 50  0000 R CNN
-F 2 "" H 8300 3150 50  0001 C CNN
+F 2 "Capacitor_SMD:C_0805_2012Metric_Pad1.18x1.45mm_HandSolder" H 8300 3150 50  0001 C CNN
 F 3 "~" H 8300 3150 50  0001 C CNN
 	1    8300 3150
@@
 F 0 "C4-0.1" H 8558 3104 50  0000 R CNN
 F 1 "0.1uF" H 8558 3195 50  0000 R CNN
-F 2 "" H 8650 3150 50  0001 C CNN
+F 2 "Capacitor_SMD:C_0805_2012Metric_Pad1.18x1.45mm_HandSolder" H 8650 3150 50  0001 C CNN
 F 3 "~" H 8650 3150 50  0001 C CNN
 	1    8650 3150
@@
 F 0 "C5-10" H 8908 3104 50  0000 R CNN
 F 1 "10uF" H 8908 3195 50  0000 R CNN
-F 2 "" H 9000 3150 50  0001 C CNN
+F 2 "Capacitor_SMD:C_0805_2012Metric_Pad1.18x1.45mm_HandSolder" H 9000 3150 50  0001 C CNN
 F 3 "~" H 9000 3150 50  0001 C CNN
 	1    9000 3150
@@
 Connection ~ 8300 3250
 Wire Wire Line
-	8500 3050 8500 2850
+	8500 3050 8500 2900
 Connection ~ 8500 3050
 Wire Wire Line
@@
 	2250 2950 2900 2950
 $Comp
-L Device:Crystal_GND24_Small Y?
+L Device:Crystal_GND24_Small Xtal1
 U 1 1 61EB290C
 P 2250 2450
-F 0 "Y?" V 2204 2594 50  0000 L CNN
+F 0 "Xtal1" V 2204 2594 50  0000 L CNN
 F 1 "16MHz" V 2295 2594 50  0000 L CNN
-F 2 "" H 2250 2450 50  0001 C CNN
+F 2 "Crystal:Crystal_SMD_3225-4Pin_3.2x2.5mm" H 2250 2450 50  0001 C CNN
 F 3 "~" H 2250 2450 50  0001 C CNN
 	1    2250 2450
@@
 F 0 "C6-22" V 1721 2250 50  0000 C CNN
 F 1 "22pF" V 1812 2250 50  0000 C CNN
-F 2 "" H 1950 2250 50  0001 C CNN
+F 2 "Capacitor_SMD:C_0805_2012Metric_Pad1.18x1.45mm_HandSolder" H 1950 2250 50  0001 C CNN
 F 3 "~" H 1950 2250 50  0001 C CNN
 	1    1950 2250
@@
 F 0 "C7-22" V 1721 2650 50  0000 C CNN
 F 1 "22pF" V 1812 2650 50  0000 C CNN
-F 2 "" H 1950 2650 50  0001 C CNN
+F 2 "Capacitor_SMD:C_0805_2012Metric_Pad1.18x1.45mm_HandSolder" H 1950 2650 50  0001 C CNN
 F 3 "~" H 1950 2650 50  0001 C CNN
 	1    1950 2650
@@
 Connection ~ 2250 2550
 $Comp
-L Switch:SW_Push SW?
+L Switch:SW_Push SW1
 U 1 1 61EBFAD8
 P 2600 2150
-F 0 "SW?" H 2600 2435 50  0000 C CNN
+F 0 "SW1" H 2600 2435 50  0000 C CNN
 F 1 "SW_Push" H 2600 2344 50  0000 C CNN
-F 2 "" H 2600 2350 50  0001 C CNN
+F 2 "Button_Switch_SMD:SW_SPST_TL3342" H 2600 2350 50  0001 C CNN
 F 3 "~" H 2600 2350 50  0001 C CNN
 	1    2600 2150
@@
 F 0 "R4-10" H 2909 1846 50  0000 L CNN
 F 1 "10k" H 2909 1755 50  0000 L CNN
-F 2 "" H 2850 1800 50  0001 C CNN
+F 2 "Resistor_SMD:R_0805_2012Metric_Pad1.20x1.40mm_HandSolder" H 2850 1800 50  0001 C CNN
 F 3 "~" H 2850 1800 50  0001 C CNN
 	1    2850 1800
@@
 Text GLabel 1800 3250 0    50   Input ~ 0
 D-
-$Comp
-L MCU_Microchip_ATmega:ATmega32U4-AU U?
-U 1 1 61E973F6
-P 3500 3650
-F 0 "U?" H 3500 1761 50  0000 C CNN
-F 1 "ATmega32U4-AU" H 3500 1670 50  0000 C CNN
-F 2 "Package_QFP:TQFP-44_10x10mm_P0.8mm" H 3500 3650 50  0001 C CIN
-F 3 "http://ww1.microchip.com/downloads/en/DeviceDoc/Atmel-7766-8-bit-AVR-ATmega16U4-32U4_Datasheet.pdf" H 3500 3650 50  0001 C CNN
-	1    3500 3650
-	1    0    0    -1
-$EndComp
-NoConn ~ 4100 4350
 NoConn ~ 2900 2750
 $Comp
-L Connector:AVR-ISP-6 J?
+L Connector:AVR-ISP-6 J1
 U 1 1 61EC9956
 P 6500 2350
-F 0 "J?" H 6171 2446 50  0000 R CNN
+F 0 "J1" H 6171 2446 50  0000 R CNN
 F 1 "AVR-ISP-6" H 6171 2355 50  0000 R CNN
-F 2 "" V 6250 2400 50  0001 C CNN
+F 2 "random-keyboard-parts:Reset_Pretty" V 6250 2400 50  0001 C CNN
 F 3 " ~" H 5225 1800 50  0001 C CNN
 	1    6500 2350
@@
 Text GLabel 6900 2450 2    50   Input ~ 0
 RESET
-Text GLabel 4100 2250 2    50   Input ~ 0
+Text GLabel 4500 2250 2    50   Input ~ 0
 SCK
-Text GLabel 4100 2350 2    50   Input ~ 0
+Text GLabel 4500 2350 2    50   Input ~ 0
 MOSI
-Text GLabel 4100 2450 2    50   Input ~ 0
+Text GLabel 4500 2450 2    50   Input ~ 0
 MISO
 $Comp
-L Type-C:HRO-TYPE-C-31-M-12 USB?
+L Type-C:HRO-TYPE-C-31-M-12 USB-C1
 U 1 1 61ECFFED
 P 6450 4500
-F 0 "USB?" H 6283 5297 60  0000 C CNN
+F 0 "USB-C1" H 6283 5297 60  0000 C CNN
 F 1 "HRO-TYPE-C-31-M-12" H 6283 5191 60  0000 C CNN
-F 2 "" H 6450 4500 60  0001 C CNN
+F 2 "Type-C:HRO-TYPE-C-31-M-12-HandSoldering" H 6450 4500 60  0001 C CNN
 F 3 "" H 6450 4500 60  0001 C CNN
 	1    6450 4500
@@
 $EndComp
 $Comp
-L Device:Polyfuse_Small F
+L Device:Polyfuse_Small F1
 U 1 1 61ED815D
 P 7300 4050
-F 0 "F" V 7095 4050 50  0000 C CNN
+F 0 "F1" V 7095 4050 50  0000 C CNN
 F 1 "500m" V 7186 4050 50  0000 C CNN
-F 2 "" H 7350 3850 50  0001 L CNN
+F 2 "Fuse:Fuse_1206_3216Metric_Pad1.42x1.75mm_HandSolder" H 7350 3850 50  0001 L CNN
 F 3 "~" H 7300 4050 50  0001 C CNN
 	1    7300 4050
@@
 	6550 4050 6650 4050
 Wire Wire Line
-	6950 4050 7200 4050
+	6950 4050 7100 4050
 Connection ~ 6950 4050
-Wire Wire Line
-	7400 4050 7700 4050
 Wire Wire Line
 	6650 4050 6650 4950
@@
 F 0 "R5-5.1" H 6909 4996 50  0000 L CNN
 F 1 "5.1k" H 6909 4905 50  0000 L CNN
-F 2 "" H 6850 4950 50  0001 C CNN
+F 2 "Resistor_SMD:R_0805_2012Metric_Pad1.20x1.40mm_HandSolder" H 6850 4950 50  0001 C CNN
 F 3 "~" H 6850 4950 50  0001 C CNN
 	1    6850 4950
@@
 F 0 "R6-5.1" H 7109 4996 50  0000 L CNN
 F 1 "5.1k" H 7109 4905 50  0000 L CNN
-F 2 "" H 7050 4950 50  0001 C CNN
+F 2 "Resistor_SMD:R_0805_2012Metric_Pad1.20x1.40mm_HandSolder" H 7050 4950 50  0001 C CNN
 F 3 "~" H 7050 4950 50  0001 C CNN
 	1    7050 4950
@@
 $EndComp
 $Comp
-L random-keyboard-parts:PRTR5V0U2X U?
+L random-keyboard-parts:PRTR5V0U2X esd1
 U 1 1 61EF2031
 P 7850 5000
-F 0 "U?" H 7850 4713 60  0000 C CNN
+F 0 "esd1" H 7850 4713 60  0000 C CNN
 F 1 "PRTR5V0U2X" H 7850 4819 60  0000 C CNN
-F 2 "" H 7850 5000 60  0001 C CNN
+F 2 "random-keyboard-parts:SOT143B" H 7850 5000 60  0001 C CNN
 F 3 "" H 7850 5000 60  0001 C CNN
 	1    7850 5000
@@
 	6700 5050 6850 5050
 $Comp
-L keyboard_parts:GND #PWR?
+L keyboard_parts:GND #PWR0115
 U 1 1 61EFFBF0
 P 6700 5300
-F 0 "#PWR?" H 6700 5350 20  0001 C CNN
+F 0 "#PWR0115" H 6700 5350 20  0001 C CNN
 F 1 "GND" H 6700 5359 30  0000 C CNN
 F 2 "" H 6700 5300 60  0000 C CNN
@@
 Connection ~ 6700 5150
 $Comp
-L power:VCC #PWR?
+L power:VCC #PWR0116
 U 1 1 61F023BC
 P 7400 5050
-F 0 "#PWR?" H 7400 4900 50  0001 C CNN
+F 0 "#PWR0116" H 7400 4900 50  0001 C CNN
 F 1 "VCC" H 7415 5223 50  0000 C CNN
 F 2 "" H 7400 5050 50  0001 C CNN
@@
 F1 "matrix.sch" 50
 $EndSheet
+Text GLabel 4100 2150 2    50   Input ~ 0
+col7
+Text GLabel 4100 2550 2    50   Input ~ 0
+col0
+Text GLabel 4100 2650 2    50   Input ~ 0
+col1
+Text GLabel 4100 2750 2    50   Input ~ 0
+col2
+Wire Wire Line
+	4100 2250 4500 2250
+Wire Wire Line
+	4100 2350 4500 2350
+Wire Wire Line
+	4500 2450 4100 2450
+NoConn ~ 4100 2850
+Text GLabel 4100 3050 2    50   Input ~ 0
+col3
+Text GLabel 4100 3150 2    50   Input ~ 0
+col4
+$Comp
+L MCU_Microchip_ATmega:ATmega32U4-AU 32U4
+U 1 1 61E973F6
+P 3500 3650
+F 0 "32U4" H 3500 1761 50  0000 C CNN
+F 1 "ATmega32U4-AU" H 3500 1670 50  0000 C CNN
+F 2 "Package_QFP:TQFP-44_10x10mm_P0.8mm" H 3500 3650 50  0001 C CIN
+F 3 "http://ww1.microchip.com/downloads/en/DeviceDoc/Atmel-7766-8-bit-AVR-ATmega16U4-32U4_Datasheet.pdf" H 3500 3650 50  0001 C CNN
+	1    3500 3650
+	1    0    0    -1
+$EndComp
+NoConn ~ 4100 3350
+Text GLabel 4100 3450 2    50   Input ~ 0
+col8
+Text GLabel 4100 3550 2    50   Input ~ 0
+col9
+Text GLabel 4100 3650 2    50   Input ~ 0
+col10
+Text GLabel 4100 3750 2    50   Input ~ 0
+col11
+Text GLabel 4100 3850 2    50   Input ~ 0
+col12
+Text GLabel 4100 3950 2    50   Input ~ 0
+col13
+Text GLabel 4100 4050 2    50   Input ~ 0
+col14
+Text GLabel 4100 4350 2    50   Input ~ 0
+row0
+Text GLabel 4100 4550 2    50   Input ~ 0
+row2
+Text GLabel 4100 4650 2    50   Input ~ 0
+row3
+Text GLabel 4100 4750 2    50   Input ~ 0
+row4
+Text GLabel 4100 4850 2    50   Input ~ 0
+row1
+Text GLabel 4100 4950 2    50   Input ~ 0
+col5
+Text GLabel 4100 5050 2    50   Input ~ 0
+col6
+Text GLabel 2850 2150 3    50   Input ~ 0
+RESET
+$Comp
+L power:PWR_FLAG #FLG0102
+U 1 1 621F2683
+P 8500 2900
+F 0 "#FLG0102" H 8500 2975 50  0001 C CNN
+F 1 "PWR_FLAG" V 8500 3028 50  0000 L CNN
+F 2 "" H 8500 2900 50  0001 C CNN
+F 3 "~" H 8500 2900 50  0001 C CNN
+	1    8500 2900
+	0    1    1    0
+$EndComp
+Connection ~ 8500 2900
+Wire Wire Line
+	8500 2900 8500 2850
+$Comp
+L power:PWR_FLAG #FLG0103
+U 1 1 621F3707
+P 7100 4050
+F 0 "#FLG0103" H 7100 4125 50  0001 C CNN
+F 1 "PWR_FLAG" H 7100 4223 50  0000 C CNN
+F 2 "" H 7100 4050 50  0001 C CNN
+F 3 "~" H 7100 4050 50  0001 C CNN
+	1    7100 4050
+	1    0    0    -1
+$EndComp
+Connection ~ 7100 4050
+Wire Wire Line
+	7100 4050 7200 4050
+Wire Wire Line
+	7400 4050 7700 4050
 $EndSCHEMATC

Commit message: pcb alignment
Connections:
- net +5V: no longer 32U4.15 (GND), 32U4.23 (GND), 32U4.35 (GND), 32U4.43 (GND), 32U4.5 (UGND), C1-1.2, C2-0.1.1, C3-0.1.1, C4-0.1.1, C5-10.1, C6-22.2, C7-22.2, J1.6 (GND), R5-5.1.2, R6-5.1.2, SW1.1, USB-C1.1 (GND), USB-C1.12 (GND), USB-C1.13 (SHIELD), Xtal1.2, Xtal1.4, esd1.1 (GND)
- new net GND: 32U4.15 (GND), 32U4.23 (GND), 32U4.35 (GND), 32U4.43 (GND), 32U4.5 (UGND), C1-1.2, C2-0.1.1, C3-0.1.1, C4-0.1.1, C5-10.1, C6-22.2, C7-22.2, J1.6 (GND), R5-5.1.2, R6-5.1.2, SW1.1, USB-C1.1 (GND), USB-C1.12 (GND), USB-C1.13 (SHIELD), Xtal1.2, Xtal1.4, esd1.1 (GND)
Changed lines of the file:
@@
 	3400 1850 3400 1700
 Connection ~ 3400 1850
-$Comp
-L keyboard_parts:GND #PWR0102
-U 1 1 61E99B0D
-P 3050 5450
-F 0 "#PWR0102" H 3050 5500 20  0001 C CNN
-F 1 "GND" H 3050 5509 30  0000 C CNN
-F 2 "" H 3050 5450 60  0000 C CNN
-F 3 "" H 3050 5450 60  0000 C CNN
-	1    3050 5450
-	1    0    0    -1
-$EndComp
 Wire Wire Line
 	3500 5450 3400 5450
@@
 F 3 "~" H 2350 3550 50  0001 C CNN
 	1    2350 3550
-	1    0    0    -1
-$EndComp
-$Comp
-L keyboard_parts:GND #PWR0104
-U 1 1 61EA46C1
-P 2350 3800
-F 0 "#PWR0104" H 2350 3850 20  0001 C CNN
-F 1 "GND" H 2350 3859 30  0000 C CNN
-F 2 "" H 2350 3800 60  0000 C CNN
-F 3 "" H 2350 3800 60  0000 C CNN
-	1    2350 3800
 	1    0    0    -1
 $EndComp
@@
 	1    0    0    -1
 $EndComp
-$Comp
-L keyboard_parts:GND #PWR0106
-U 1 1 61EAE9F7
-P 8500 3450
-F 0 "#PWR0106" H 8500 3500 20  0001 C CNN
-F 1 "GND" H 8500 3509 30  0000 C CNN
-F 2 "" H 8500 3450 60  0000 C CNN
-F 3 "" H 8500 3450 60  0000 C CNN
-	1    8500 3450
-	1    0    0    -1
-$EndComp
 Wire Wire Line
 	7950 3050 8300 3050
@@
 Wire Wire Line
 	8500 3050 8650 3050
-Wire Wire Line
-	8500 3250 8500 3450
 Connection ~ 8500 3250
 Wire Wire Line
@@
 	0    1    1    0
 $EndComp
-$Comp
-L keyboard_parts:GND #PWR0108
-U 1 1 61EBA72E
-P 1850 2800
-F 0 "#PWR0108" H 1850 2850 20  0001 C CNN
-F 1 "GND" H 1850 2859 30  0000 C CNN
-F 2 "" H 1850 2800 60  0000 C CNN
-F 3 "" H 1850 2800 60  0000 C CNN
-	1    1850 2800
-	1    0    0    -1
-$EndComp
 Wire Wire Line
 	2250 2350 2050 2350
@@
 Wire Wire Line
 	2150 2800 1850 2800
-Connection ~ 1850 2800
 Wire Wire Line
 	2350 2450 2350 2700
@@
 	1    0    0    -1
 $EndComp
-$Comp
-L keyboard_parts:GND #PWR0109
-U 1 1 61EC0936
-P 2250 2100
-F 0 "#PWR0109" H 2250 2150 20  0001 C CNN
-F 1 "GND" H 2250 2159 30  0000 C CNN
-F 2 "" H 2250 2100 60  0000 C CNN
-F 3 "" H 2250 2100 60  0000 C CNN
-	1    2250 2100
-	1    0    0    -1
-$EndComp
 Wire Wire Line
 	2900 2150 2850 2150
 Wire Wire Line
 	2400 2150 2400 2100
-Wire Wire Line
-	2400 2100 2250 2100
 $Comp
 L Device:R_Small R4-10
@@
 F 3 " ~" H 5225 1800 50  0001 C CNN
 	1    6500 2350
-	1    0    0    -1
-$EndComp
-$Comp
-L keyboard_parts:GND #PWR0111
-U 1 1 61ECC37C
-P 6400 2750
-F 0 "#PWR0111" H 6400 2800 20  0001 C CNN
-F 1 "GND" H 6400 2809 30  0000 C CNN
-F 2 "" H 6400 2750 60  0000 C CNN
-F 3 "" H 6400 2750 60  0000 C CNN
-	1    6400 2750
 	1    0    0    -1
 $EndComp
@@
 Wire Wire Line
 	6700 5050 6850 5050
-$Comp
-L keyboard_parts:GND #PWR0115
-U 1 1 61EFFBF0
-P 6700 5300
-F 0 "#PWR0115" H 6700 5350 20  0001 C CNN
-F 1 "GND" H 6700 5359 30  0000 C CNN
-F 2 "" H 6700 5300 60  0000 C CNN
-F 3 "" H 6700 5300 60  0000 C CNN
-	1    6700 5300
-	1    0    0    -1
-$EndComp
-Wire Wire Line
-	6700 5150 6700 5300
 Connection ~ 6700 5150
 $Comp
@@
 Wire Wire Line
 	7400 4050 7700 4050
+Wire Wire Line
+	6700 5150 6700 5300
+Wire Wire Line
+	2250 2100 2400 2100
+Wire Wire Line
+	8500 3250 8500 3450
+$Comp
+L power:GND #PWR?
+U 1 1 62479121
+P 8500 3450
+F 0 "#PWR?" H 8500 3200 50  0001 C CNN
+F 1 "GND" H 8505 3277 50  0000 C CNN
+F 2 "" H 8500 3450 50  0001 C CNN
+F 3 "" H 8500 3450 50  0001 C CNN
+	1    8500 3450
+	1    0    0    -1
+$EndComp
+$Comp
+L power:GND #PWR?
+U 1 1 6247C0CA
+P 2250 2100
+F 0 "#PWR?" H 2250 1850 50  0001 C CNN
+F 1 "GND" H 2255 1927 50  0000 C CNN
+F 2 "" H 2250 2100 50  0001 C CNN
+F 3 "" H 2250 2100 50  0001 C CNN
+	1    2250 2100
+	1    0    0    -1
+$EndComp
+$Comp
+L power:GND #PWR?
+U 1 1 6247D056
+P 1850 2800
+F 0 "#PWR?" H 1850 2550 50  0001 C CNN
+F 1 "GND" H 1855 2627 50  0000 C CNN
+F 2 "" H 1850 2800 50  0001 C CNN
+F 3 "" H 1850 2800 50  0001 C CNN
+	1    1850 2800
+	1    0    0    -1
+$EndComp
+Connection ~ 1850 2800
+$Comp
+L power:GND #PWR?
+U 1 1 6247E214
+P 2350 3800
+F 0 "#PWR?" H 2350 3550 50  0001 C CNN
+F 1 "GND" H 2355 3627 50  0000 C CNN
+F 2 "" H 2350 3800 50  0001 C CNN
+F 3 "" H 2350 3800 50  0001 C CNN
+	1    2350 3800
+	1    0    0    -1
+$EndComp
+$Comp
+L power:GND #PWR?
+U 1 1 6247EC26
+P 3050 5450
+F 0 "#PWR?" H 3050 5200 50  0001 C CNN
+F 1 "GND" H 3055 5277 50  0000 C CNN
+F 2 "" H 3050 5450 50  0001 C CNN
+F 3 "" H 3050 5450 50  0001 C CNN
+	1    3050 5450
+	1    0    0    -1
+$EndComp
+$Comp
+L power:GND #PWR?
+U 1 1 6247EF75
+P 6700 5300
+F 0 "#PWR?" H 6700 5050 50  0001 C CNN
+F 1 "GND" H 6705 5127 50  0000 C CNN
+F 2 "" H 6700 5300 50  0001 C CNN
+F 3 "" H 6700 5300 50  0001 C CNN
+	1    6700 5300
+	1    0    0    -1
+$EndComp
+$Comp
+L power:GND #PWR?
+U 1 1 6247FB74
+P 6400 2750
+F 0 "#PWR?" H 6400 2500 50  0001 C CNN
+F 1 "GND" H 6405 2577 50  0000 C CNN
+F 2 "" H 6400 2750 50  0001 C CNN
+F 3 "" H 6400 2750 50  0001 C CNN
+	1    6400 2750
+	1    0    0    -1
+$EndComp
 $EndSCHEMATC

Commit message: switch matrix routing
Changed lines of the file:
@@
 	8500 3250 8500 3450
 $Comp
-L power:GND #PWR?
+L power:GND #PWR0102
 U 1 1 62479121
 P 8500 3450
-F 0 "#PWR?" H 8500 3200 50  0001 C CNN
+F 0 "#PWR0102" H 8500 3200 50  0001 C CNN
 F 1 "GND" H 8505 3277 50  0000 C CNN
 F 2 "" H 8500 3450 50  0001 C CNN
@@
 $EndComp
 $Comp
-L power:GND #PWR?
+L power:GND #PWR0104
 U 1 1 6247C0CA
 P 2250 2100
-F 0 "#PWR?" H 2250 1850 50  0001 C CNN
+F 0 "#PWR0104" H 2250 1850 50  0001 C CNN
 F 1 "GND" H 2255 1927 50  0000 C CNN
 F 2 "" H 2250 2100 50  0001 C CNN
@@
 $EndComp
 $Comp
-L power:GND #PWR?
+L power:GND #PWR0106
 U 1 1 6247D056
 P 1850 2800
-F 0 "#PWR?" H 1850 2550 50  0001 C CNN
+F 0 "#PWR0106" H 1850 2550 50  0001 C CNN
 F 1 "GND" H 1855 2627 50  0000 C CNN
 F 2 "" H 1850 2800 50  0001 C CNN
@@
 Connection ~ 1850 2800
 $Comp
-L power:GND #PWR?
+L power:GND #PWR0108
 U 1 1 6247E214
 P 2350 3800
-F 0 "#PWR?" H 2350 3550 50  0001 C CNN
+F 0 "#PWR0108" H 2350 3550 50  0001 C CNN
 F 1 "GND" H 2355 3627 50  0000 C CNN
 F 2 "" H 2350 3800 50  0001 C CNN
@@
 $EndComp
 $Comp
-L power:GND #PWR?
+L power:GND #PWR0109
 U 1 1 6247EC26
 P 3050 5450
-F 0 "#PWR?" H 3050 5200 50  0001 C CNN
+F 0 "#PWR0109" H 3050 5200 50  0001 C CNN
 F 1 "GND" H 3055 5277 50  0000 C CNN
 F 2 "" H 3050 5450 50  0001 C CNN
@@
 $EndComp
 $Comp
-L power:GND #PWR?
+L power:GND #PWR0111
 U 1 1 6247EF75
 P 6700 5300
-F 0 "#PWR?" H 6700 5050 50  0001 C CNN
+F 0 "#PWR0111" H 6700 5050 50  0001 C CNN
 F 1 "GND" H 6705 5127 50  0000 C CNN
 F 2 "" H 6700 5300 50  0001 C CNN
@@
 $EndComp
 $Comp
-L power:GND #PWR?
+L power:GND #PWR0115
 U 1 1 6247FB74
 P 6400 2750
-F 0 "#PWR?" H 6400 2500 50  0001 C CNN
+F 0 "#PWR0115" H 6400 2500 50  0001 C CNN
 F 1 "GND" H 6405 2577 50  0000 C CNN
 F 2 "" H 6400 2750 50  0001 C CNN
@@
 	1    0    0    -1
 $EndComp
+Text GLabel 7300 4550 1    50   Input ~ 0
+DN
+Text GLabel 7300 4650 3    50   Input ~ 0
+DP
 $EndSCHEMATC
